Commit message: c12 for cos(q1+q3)

File: robots/simple/rrrp.urdf (robot description, URDF)
Before this commit: robot rrrp, 10 links, 9 joints
Links:
- removed link end_effector
- added link tool0; visual sphere radius=.005
Joints:
- joint joint3: type fixed -> revolute
- joint joint4: origin xyz=0. -0.07 0.0 rpy=1.5707963267948 0 0 -> xyz=0. 0 0.0 rpy=1.5707963267948 0 0
- joint link4_2: child end_effector -> tool0; origin xyz=0.0 0 0.0 rpy=0 0 0 -> xyz=0.0 0.0 0.07 rpy=0 0 0
